File: Mmuo.kicad_pcb (KiCad board)
At the start: 2 copper layers, 0 parts

Commit message: Schematics Verifcation
Other:
- copper layers 2 -> 4
Changed lines of the file:
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@@
 	(generator_version "9.0")
 	(general
-		(thickness 1.5982)
+		(thickness 1.5842)
 		(legacy_teardrops no)
 	)
@@
 	(layers
 		(0 "F.Cu" signal)
+		(4 "In1.Cu" signal)
+		(6 "In2.Cu" signal)
 		(2 "B.Cu" signal)
+		(9 "F.Adhes" user "F.Adhesive")
 		(11 "B.Adhes" user "B.Adhesive")
 		(13 "F.Paste" user)
@@
 		(31 "F.CrtYd" user "F.Courtyard")
 		(29 "B.CrtYd" user "B.Courtyard")
-		(33 "B.Fab" user)
 	)
 	(setup
@@
 			(layer "F.Mask"
 				(type "Top Solder Mask")
-				(thickness 0.017)
+				(thickness 0.01)
 			)
 			(layer "F.Cu"
@@
 			)
 			(layer "dielectric 1"
-				(type "core")
-				(thickness 1.4942)
+				(type "prepreg")
+				(color "FR4 natural")
+				(thickness 0.0994)
 				(material "3313")
 				(epsilon_r 4.2)
+				(loss_tangent 0)
+			)
+			(layer "In1.Cu"
+				(type "copper")
+				(thickness 0.0152)
+			)
+			(layer "dielectric 2"
+				(type "core")
+				(thickness 1.265)
+				(material "FR4")
+				(epsilon_r 4.2)
 				(loss_tangent 0.02)
+			)
+			(layer "In2.Cu"
+				(type "copper")
+				(thickness 0.0152)
+			)
+			(layer "dielectric 3"
+				(type "prepreg")
+				(color "FR4 natural")
+				(thickness 0.0994)
+				(material "3313")
+				(epsilon_r 4.2)
+				(loss_tangent 0)
 			)
 			(layer "B.Cu"
@@
 			(layer "B.Mask"
 				(type "Bottom Solder Mask")
-				(thickness 0.017)
+				(thickness 0.01)
 			)
 			(layer "B.Paste"
@@
 				(type "Bottom Silk Screen")
 			)
-			(copper_finish "HAL lead-free")
-			(dielectric_constraints no)
+			(copper_finish "None")
+			(dielectric_constraints yes)
 		)
 		(pad_to_mask_clearance 0)
@@
 	)
 	(net 0 "")
-	(net 1 "/Vss")
 	(zone
-		(net 1)
-		(net_name "/Vss")
+		(net 0)
+		(net_name "")
 		(layer "B.Cu")
 		(name "$teardrop_padvia$")

Commit message: replacing 3v3 LDO to boost-buck converter
Parts:
- added AE1: AMCA31-2R450G-S1F-T3, AMCA31-2R450G-S1F-T3:ANTC3216X140N, F.Cu at (197.3, 98.6)
- added AE2: MLPF-WB55-01E3, MLPF-WB55-01E3:MLPF-WB55-01E3_STM, F.Cu at (189.4, 99.8)
- added C1: 1u, Capacitor_SMD:C_0603_1608Metric_Pad1.08x0.95mm_HandSolder, F.Cu at (117.3, 94.0)
- added C10: 1u, Capacitor_SMD:C_0603_1608Metric_Pad1.08x0.95mm_HandSolder, B.Cu at (139.3, 110.9)
- added C11: 1u, Capacitor_SMD:C_0603_1608Metric_Pad1.08x0.95mm_HandSolder, B.Cu at (146.6, 110.9)
- added C12: 1u, Capacitor_SMD:C_0603_1608Metric_Pad1.08x0.95mm_HandSolder, B.Cu at (138.4, 112.8)
- added C13: 1u, Capacitor_SMD:C_0603_1608Metric_Pad1.08x0.95mm_HandSolder, B.Cu at (147.3, 112.7)
- added C14: 1u, Capacitor_SMD:C_0603_1608Metric_Pad1.08x0.95mm_HandSolder, B.Cu at (146.9, 114.5)
- added C15: 4u7, Capacitor_SMD:C_0805_2012Metric_Pad1.18x1.45mm_HandSolder, B.Cu at (142.9, 109.0)
- added C16: 1u, Capacitor_SMD:C_0603_1608Metric_Pad1.08x0.95mm_HandSolder, B.Cu at (127.4, 106.5)
- added C17: x, Capacitor_SMD:C_0603_1608Metric_Pad1.08x0.95mm_HandSolder, F.Cu at (149.4, 120.4)
- added C18: x, Capacitor_SMD:C_0603_1608Metric_Pad1.08x0.95mm_HandSolder, F.Cu at (150.0, 115.2)
- added C19: 0u1, Capacitor_SMD:C_0603_1608Metric_Pad1.08x0.95mm_HandSolder, F.Cu at (176.8, 108.6)
- added C2: 2u2, Capacitor_SMD:C_0603_1608Metric_Pad1.08x0.95mm_HandSolder, F.Cu at (125.4, 94.3)
- added C20: 0u1, Capacitor_SMD:C_0603_1608Metric_Pad1.08x0.95mm_HandSolder, F.Cu at (186.2, 102.1)
- added C21: 0u1, Capacitor_SMD:C_0603_1608Metric_Pad1.08x0.95mm_HandSolder, F.Cu at (180.3, 107.8)
- added C22: 0u1, Capacitor_SMD:C_0603_1608Metric_Pad1.08x0.95mm_HandSolder, F.Cu at (186.2, 98.5)
- added C23: 0u1, Capacitor_SMD:C_0603_1608Metric_Pad1.08x0.95mm_HandSolder, F.Cu at (172.2, 104.0)
- added C24: 0u1, Capacitor_SMD:C_0603_1608Metric_Pad1.08x0.95mm_HandSolder, F.Cu at (171.4, 100.0)
- added C25: 0u1, Capacitor_SMD:C_0603_1608Metric_Pad1.08x0.95mm_HandSolder, F.Cu at (174.6, 93.6)
- added C26: 0u1, Capacitor_SMD:C_0603_1608Metric_Pad1.08x0.95mm_HandSolder, F.Cu at (176.1, 93.6)
- added C27: 4u7, Capacitor_SMD:C_0805_2012Metric_Pad1.18x1.45mm_HandSolder, F.Cu at (186.7, 109.5)
- added C28: 0u1, Capacitor_SMD:C_0603_1608Metric_Pad1.08x0.95mm_HandSolder, F.Cu at (158.4, 94.5)
- added C29: 0u1, Capacitor_SMD:C_0603_1608Metric_Pad1.08x0.95mm_HandSolder, F.Cu at (193.2, 118.6)
- added C3: 1u, Capacitor_SMD:C_0603_1608Metric_Pad1.08x0.95mm_HandSolder, B.Cu at (138.2, 115.6)
- added C30: 4u7, Capacitor_SMD:C_0805_2012Metric_Pad1.18x1.45mm_HandSolder, F.Cu at (181.7, 93.1)
- added C31: 0u1, Capacitor_SMD:C_0603_1608Metric_Pad1.08x0.95mm_HandSolder, F.Cu at (163.4, 104.8)
- added C32: 1p2, Capacitor_SMD:C_0402_1005Metric, F.Cu at (191.4, 98.9)
- added C33: 1p2, Capacitor_SMD:C_0402_1005Metric, F.Cu at (193.6, 99.0)
- added C34: 10p, Capacitor_SMD:C_0603_1608Metric_Pad1.08x0.95mm_HandSolder, F.Cu at (175.0, 107.7)
- added C35: 10p, Capacitor_SMD:C_0603_1608Metric_Pad1.08x0.95mm_HandSolder, F.Cu at (171.1, 107.7)
- added C36: 0u1, Capacitor_SMD:C_0603_1608Metric_Pad1.08x0.95mm_HandSolder, F.Cu at (178.4, 115.4)
- added C37: 0u1, Capacitor_SMD:C_0603_1608Metric_Pad1.08x0.95mm_HandSolder, F.Cu at (183.7, 113.0)
- added C4: 33n, Capacitor_SMD:C_0603_1608Metric_Pad1.08x0.95mm_HandSolder, F.Cu at (127.2, 96.9)
- added C5: 1u, Capacitor_SMD:C_0603_1608Metric_Pad1.08x0.95mm_HandSolder, F.Cu at (134.6, 103.4)
- added C6: 1u, Capacitor_SMD:C_0603_1608Metric_Pad1.08x0.95mm_HandSolder, F.Cu at (134.6, 96.6)
- added C7: 22u, Capacitor_SMD:C_0603_1608Metric_Pad1.08x0.95mm_HandSolder, F.Cu at (128.7, 101.7)
- added C8: 1u, Capacitor_SMD:C_0603_1608Metric_Pad1.08x0.95mm_HandSolder, F.Cu at (137.5, 94.6)
- added C9: 1u, Capacitor_SMD:C_0603_1608Metric_Pad1.08x0.95mm_HandSolder, F.Cu at (142.5, 98.8)
- added D1: LED, LED_SMD:LED_0805_2012Metric_Pad1.15x1.40mm_HandSolder, F.Cu at (132.7, 93.0)
- added D2: LED, LED_SMD:LED_0805_2012Metric_Pad1.15x1.40mm_HandSolder, F.Cu at (112.7, 112.1)
- added D3: LED, LED_SMD:LED_0805_2012Metric_Pad1.15x1.40mm_HandSolder, F.Cu at (119.0, 113.2)
- added D4: D_Schottky, Diode_SMD:D_SOD-123, F.Cu at (158.7, 92.1)
- added D5: D_Schottky, Diode_SMD:D_SOD-123, F.Cu at (159.5, 111.3)
- added D6: LED, LED_SMD:LED_0805_2012Metric_Pad1.15x1.40mm_HandSolder, F.Cu at (171.4, 125.0)
- added D7: LED, LED_SMD:LED_0805_2012Metric_Pad1.15x1.40mm_HandSolder, F.Cu at (174.4, 125.0)
- added D8: LED, LED_SMD:LED_0805_2012Metric_Pad1.15x1.40mm_HandSolder, F.Cu at (177.4, 125.0)
- added IC1: A121-001-T&R, A121-001-T&R:A121001TR, F.Cu at (143.0, 113.5)
- added IC2: BQ24253RGER, BQ24253RGER:QFN50P400X400X100-25N-D, F.Cu at (122.8, 98.9)
- added IC3: ADPL40502AUJZ-1.8-R7, ADPL40502AUJZ-1.8-R7:SOT95P280X100-5N, F.Cu at (139.5, 98.7)
- added J1: USB_C_Receptacle_USB2.0_16P, Connector_USB:USB_C_Receptacle_GCT_USB4105-xx-A_16P_TopMnt_Horizontal, F.Cu at (103.4, 99.7)
- added J2: B2B-PH-K-S, B2B_PH_K_S:JST_B2B-PH-K-S, B.Cu at (129.1, 111.4)
- added J3: SW_Debug, Connector:Tag-Connect_TC2030-IDC-FP_2x03_P1.27mm_Vertical, F.Cu at (167.4, 88.5)
- added L1: 1u, Inductor_SMD:L_0805_2012Metric_Pad1.05x1.20mm_HandSolder, F.Cu at (129.5, 98.9)
- added L2: 10n, Inductor_SMD:L_0805_2012Metric_Pad1.05x1.20mm_HandSolder, F.Cu at (178.0, 93.1)
- added L3: 10u, Inductor_SMD:L_0805_2012Metric_Pad1.05x1.20mm_HandSolder, F.Cu at (179.8, 93.1)
- added L4: 3n6, Inductor_SMD:L_0402_1005Metric, F.Cu at (192.5, 99.0)
- added LS1: SMT-0440-T-R, SMT-0440-T-R:SMT0440TR, F.Cu at (159.5, 115.7)
- added Q1: BSS84, Package_TO_SOT_SMD:SOT-23, F.Cu at (114.6, 106.4)
- added Q2: BSS138, Package_TO_SOT_SMD:SOT-23, F.Cu at (121.1, 107.4)
- added Q3: MMBT3904, Package_TO_SOT_SMD:SOT-23, F.Cu at (158.2, 120.6)
- added R1: 200, Resistor_SMD:R_0603_1608Metric_Pad0.98x0.95mm_HandSolder, F.Cu at (120.3, 92.8)
- added R10: 10K, Resistor_SMD:R_0603_1608Metric_Pad0.98x0.95mm_HandSolder, B.Cu at (124.3, 106.5)
- added R11: 5K, Resistor_SMD:R_0805_2012Metric_Pad1.20x1.40mm_HandSolder, F.Cu at (117.5, 106.3)
- added R12: 5K, Resistor_SMD:R_0805_2012Metric_Pad1.20x1.40mm_HandSolder, F.Cu at (123.9, 107.3)
- added R13: 620, Resistor_SMD:R_0603_1608Metric_Pad0.98x0.95mm_HandSolder, F.Cu at (113.8, 109.3)
- added R14: 620, Resistor_SMD:R_0603_1608Metric_Pad0.98x0.95mm_HandSolder, F.Cu at (120.1, 110.4)
- added R15: 10K, Resistor_SMD:R_0805_2012Metric_Pad1.20x1.40mm_HandSolder, F.Cu at (149.9, 88.0)
- added R16: 0, Resistor_SMD:R_0603_1608Metric_Pad0.98x0.95mm_HandSolder, F.Cu at (185.7, 95.9)
- added R17: 220 or 1k, Resistor_SMD:R_0603_1608Metric_Pad0.98x0.95mm_HandSolder, F.Cu at (161.0, 120.6)
- added R18: 4K7, Resistor_SMD:R_0805_2012Metric_Pad1.20x1.40mm_HandSolder, F.Cu at (154.7, 102.3)
- added R19: 4K7, Resistor_SMD:R_0805_2012Metric_Pad1.20x1.40mm_HandSolder, F.Cu at (158.1, 101.5)
- added R2: 515, Resistor_SMD:R_0603_1608Metric_Pad0.98x0.95mm_HandSolder, F.Cu at (121.9, 92.8)
- added R20: 10k, Resistor_SMD:R_0805_2012Metric_Pad1.20x1.40mm_HandSolder, F.Cu at (205.1, 122.9)
- added R21: 4K7, Resistor_SMD:R_0603_1608Metric_Pad0.98x0.95mm_HandSolder, F.Cu at (154.8, 106.1)
- added R22: 220, Resistor_SMD:R_0603_1608Metric_Pad0.98x0.95mm_HandSolder, F.Cu at (189.3, 114.8)
- added R23: 220, Resistor_SMD:R_0603_1608Metric_Pad0.98x0.95mm_HandSolder, F.Cu at (191.8, 114.8)
- added R24: 220, Resistor_SMD:R_0603_1608Metric_Pad0.98x0.95mm_HandSolder, F.Cu at (194.3, 114.8)
- added R3: 0, Resistor_SMD:R_0603_1608Metric_Pad0.98x0.95mm_HandSolder, F.Cu at (124.5, 92.7)
- added R4: 220, Resistor_SMD:R_0603_1608Metric_Pad0.98x0.95mm_HandSolder, F.Cu at (134.6, 94.9)
- added R5: 10K, Resistor_SMD:R_0805_2012Metric_Pad1.20x1.40mm_HandSolder, F.Cu at (106.2, 106.6)
- added R6: 10K, Resistor_SMD:R_0805_2012Metric_Pad1.20x1.40mm_HandSolder, F.Cu at (106.3, 92.5)
- added R7: 10K, Resistor_SMD:R_0805_2012Metric_Pad1.20x1.40mm_HandSolder, F.Cu at (117.0, 96.2)
- added R8: 10K, Resistor_SMD:R_0805_2012Metric_Pad1.20x1.40mm_HandSolder, F.Cu at (119.0, 101.7)
- added R9: 250, Resistor_SMD:R_0603_1608Metric_Pad0.98x0.95mm_HandSolder, B.Cu at (125.8, 106.5)
- added S1: PTS815, PS815_SJK:PTS815SJK250SMTRLFS, F.Cu at (183.6, 117.6)
- added SW1: PTS815, PS815_SJK:PTS815SJK250SMTRLFS, F.Cu at (174.5, 116.7)
- added U1: USBLC6-2SC6, Package_TO_SOT_SMD:SOT-23-6, F.Cu at (113.2, 99.5)
- added U2: RT9166A-33GXL, RT9166A_33GXL:VREG_AP7370-33Y-13, F.Cu at (133.8, 100.0)
- added U3: EKMB1309113K, EKMB:XDCR_EKMB, F.Cu at (150.8, 94.8)
- added U4: STM32WB55CGU6, Package_DFN_QFN:QFN-48-1EP_7x7mm_P0.5mm_EP5.6x5.6mm, F.Cu at (179.5, 101.2)
- added U5: MCP9808_MSOP, Package_SO:MSOP-8_3x3mm_P0.65mm, F.Cu at (159.2, 104.7)
- added Y1: 24MHz, Crystal:Crystal_SMD_2016-4Pin_2.0x1.6mm, F.Cu at (149.3, 118.3)
- added Y2: 32MHz, Crystal:Crystal_SMD_2016-4Pin_2.0x1.6mm, F.Cu at (186.0, 93.5)
- added Y3: 32K768, Crystal:Crystal_SMD_2012-2Pin_2.0x1.2mm_HandSoldering, F.Cu at (173.0, 107.8)

Commit message: Layout and initial routing
Parts:
- removed U2: RT9166A-33GXL, RT9166A_33GXL:VREG_AP7370-33Y-13
- added C38: 10u, Capacitor_SMD:C_0603_1608Metric_Pad1.08x0.95mm_HandSolder, F.Cu at (139.5, 102.8)
- added H1: MountingHole_Pad, MountingHole:MountingHole_3.2mm_M3_DIN965_Pad_TopBottom, F.Cu at (109.6, 85.8)
- added H2: MountingHole_Pad, MountingHole:MountingHole_3.2mm_M3_DIN965_Pad_TopBottom, F.Cu at (109.6, 123.2)
- added H3: MountingHole_Pad, MountingHole:MountingHole_3.2mm_M3_DIN965_Pad_TopBottom, F.Cu at (190.2, 123.2)
- added H4: MountingHole_Pad, MountingHole:MountingHole_3.2mm_M3_DIN965_Pad_TopBottom, F.Cu at (190.2, 85.8)
- added IC4: RAA2361052GNP#HC5, RAA2361052GNP:SON50P250X250X90-11N-D, F.Cu at (138.1, 98.6)
- added L5: 1u, Inductor_SMD:L_0805_2012Metric_Pad1.05x1.20mm_HandSolder, F.Cu at (142.8, 98.6)
- added R25: 0, Resistor_SMD:R_0603_1608Metric_Pad0.98x0.95mm_HandSolder, F.Cu at (133.6, 99.4)
- added R26: 332k, Resistor_SMD:R_0603_1608Metric_Pad0.98x0.95mm_HandSolder, F.Cu at (135.8, 101.2)
- C5, C6: value 1u -> 10u
- moved C29 43.2 mm to (163.3, 87.4)
- moved D8 38.5 mm to (180.2, 86.6), turned to 0 degrees
- moved D7 30.3 mm to (167.7, 95.5)
- moved R24 30.1 mm to (183.8, 86.6), turned to 180 degrees
- moved R20 29.8 mm to (177.1, 112.6), turned to -90 degrees
- moved R23 29.5 mm to (169.6, 95.3)
- moved R22 28.0 mm to (165.9, 99.4), turned to -90 degrees
- moved D6 26.7 mm to (164.0, 99.4), turned to -90 degrees
- moved D1 16.1 mm to (140.8, 106.9)
- moved C8 13.5 mm to (129.6, 105.5)
- moved R4 11.5 mm to (142.9, 102.8), turned to -90 degrees
- moved IC3 10.9 mm to (132.8, 107.3)
- moved C9 10.9 mm to (135.8, 107.4)
- moved C5 9.97 mm to (139.3, 94.7), turned to 90 degrees
- moved C6 9.03 mm to (141.2, 102.8), turned to -90 degrees
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Connections:
- net /USB_ESD_M renamed /USB_ESD_N
- net /USB_M renamed /USB_N
Routing:
- net +5V: track 0.00 -> 48.6 mm, vias 0 -> 2
- net Net-(IC2-SYS_1): track 0.00 -> 24.9 mm
- net Net-(IC2-BAT_1): track 0.00 -> 19.6 mm, vias 0 -> 1
- net +3V3: track 0.00 -> 12.4 mm, vias 0 -> 20
- net Net-(IC2-ISET): track 0.00 -> 11.2 mm, vias 0 -> 1
- net Net-(IC2-TS): track 0.00 -> 10.8 mm, vias 0 -> 1
- net /USB_N: track 0.00 -> 9.18 mm
- net /USB_P: track 0.00 -> 9.12 mm
- net /~{CHG}: track 0.00 -> 8.80 mm
- net /CC1: track 0.00 -> 7.46 mm
- net /~{PG}: track 0.00 -> 7.43 mm
- net /USB_ESD_P: track 0.00 -> 7.41 mm
- net /USB_ESD_N: track 0.00 -> 7.32 mm, vias 0 -> 2
- net /CC2: track 0.00 -> 7.06 mm
- net /BT: track 0.00 -> 6.49 mm
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- added copper zone on In2.Cu, net +1V8
- added copper zone on In2.Cu, net +3V3
- added copper zone on F.Cu, net /SMPSFB
- added copper zone on In1.Cu, net GND
Other:
- board outline added: 99.3 x 46.2 mm

Commit message: PCB design and full verification
Parts:
- removed C31: 0u1, Capacitor_SMD:C_0603_1608Metric_Pad1.08x0.95mm_HandSolder
- removed R18, R19: 4K7, Resistor_SMD:R_0805_2012Metric_Pad1.20x1.40mm_HandSolder
- removed R21: 4K7, Resistor_SMD:R_0603_1608Metric_Pad0.98x0.95mm_HandSolder
- removed U5: MCP9808_MSOP, Package_SO:MSOP-8_3x3mm_P0.65mm
- added G***: LOGO, Lion:Lion, F.Cu at (134.6, 89.2)
- added G***: LOGO, Lion:Lion, B.Cu at (143.4, 120.8)
- moved C21 8.38 mm to (173.1, 113.7)
- moved J2 6.61 mm to (129.1, 122.6)
- moved C27 5.14 mm to (179.8, 113.7)
- moved C20 3.03 mm to (188.3, 104.4)
- moved R20 1.48 mm to (175.8, 113.4)
- moved C18 1.23 mm to (152.3, 118.2), turned to 0 degrees
- moved C22 1.21 mm to (186.7, 96.7)
- moved Y2 1.21 mm to (187.0, 92.8)
- moved R16 1.21 mm to (186.7, 95.2)
- moved D7 1.15 mm to (168.6, 96.2)
- moved R23 1.12 mm to (170.3, 96.2)
- moved C24 1.01 mm to (170.1, 100.7)
- moved R22 0.63 mm to (166.0, 100.0)
- moved D6 0.61 mm to (164.2, 99.9)
- moved C23 0.30 mm to (170.0, 104.2)
Routing:
- net GND: track 0.00 -> 124.1 mm, vias 75 -> 129
- net /SPI_SS: track 0.00 -> 69.5 mm, vias 0 -> 2
- net /SPI_MOSI: track 0.00 -> 68.8 mm, vias 0 -> 2
- net /~{RST}: track 0.00 -> 68.5 mm
- net /SPI_MISO: track 0.00 -> 64.4 mm, vias 0 -> 2
- net /SPI_CLK: track 0.00 -> 61.0 mm, vias 0 -> 2
- net /SPI_INT: track 0.00 -> 58.6 mm, vias 0 -> 2
- net /SPI_EN: track 0.00 -> 55.6 mm, vias 0 -> 2
- net +3V3: track 12.4 -> 61.8 mm, vias 20 -> 19
- net /PIR_PA0: track 4.35 -> 50.5 mm, vias 0 -> 3
- net +5V: track 48.6 -> 82.2 mm, vias 2 -> 9
- net /Buzzer: track 0.00 -> 24.5 mm, vias 0 -> 2
- net /Pair_button: track 0.00 -> 21.8 mm
- net +1V8: track 1.83 -> 22.4 mm, vias 5 -> 8
- net /SWO: track 0.00 -> 19.5 mm
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- added copper zone on F.Cu, net GND
Other:
- board text added: "${TITLE} ${REVISION}"
- board text added: "5V @ 2A Charging"
- board text added: "Li-Po Battery Attachment"
- board text added: "Pair"
- board text added: "Power Supply"
- board text added: "Reset"
